File: eater-deluxe.kicad_pcb (KiCad board)
At the start: 2 copper layers, 214.2 x 149.5 mm, 41 parts, among them J1 PJ-202A, J2 DE9_Socket, SW1 RESET, U1 6502, U2 W65C22NxP, U3 W65C51NxP, U4 28C256, U5 HM62256BLP, U6 CD74HC00E, U7 MAX232, U8 LCD Module Connector, X1 MXO45-3C-1M000000, Y1 1.8432MHz

Commit message: fix Footprint for caps
were 10mm pitch, now they're 5mm pitch.

Signed-off-by: Lucy Mielke <user@domain.tld>
Parts:
- C10, C11, C12, C13, C14, C15, C16, C17, C18, C19, C20, C5, C6, C7, C8, C9: footprint Capacitor_THT:C_Disc_D10.5mm_W5.0mm_P10.00mm -> Capacitor_THT:C_Disc_D4.3mm_W1.9mm_P5.00mm
- moved C17 15.1 mm to (193.0, 79.8), turned to 180 degrees
- moved C11 8.36 mm to (126.5, 122.0)
- moved C12 5.46 mm to (122.5, 131.0)
- moved C7 5.18 mm to (126.4, 187.0)
- moved C18 5.02 mm to (196.0, 204.5)
- moved C6 5.00 mm to (142.5, 88.5)
- moved C5 4.93 mm to (224.5, 192.3)
- moved C9 3.89 mm to (257.0, 95.5)
- moved C19 2.50 mm to (196.0, 175.5)
- moved C20 1.95 mm to (183.5, 111.0), turned to 90 degrees
- turned C16 to 90 degrees
- turned C8 to 0 degrees
Routing:
- net Net-(U7-C2-): track 22.0 -> 11.2 mm
- net Net-(U7-C1+): track 14.3 -> 5.65 mm
- net Net-(U7-C1-): track 12.3 -> 5.63 mm
- net Net-(U7-C2+): track 14.8 -> 10.2 mm
- net /5V: track 1041.9 -> 1044.2 mm
- net Net-(U3-XTAL1): track 19.1 -> 18.2 mm
