File: eater-deluxe.kicad_sch (KiCad schematic)
At the start: 39 parts, among them J1 PJ-202A, J2 DE9_Socket, SW1 RESET, U1 6502, U2 W65C22NxP, U3 W65C51NxP, U4 28C256, U5 HM62256BLP, U6 CD74HC00E, U7 MAX232, U8 LCD Module Connector, X1 MXO45-3C-1M000000, Y1 1.8432MHz

Commit message: Correct X1 pinout, fix LCD Pins, add pullup resistors for interrupt lines
Signed-off-by: Lucy Mielke <user@domain.tld>
Parts:
- added R4, R5: 1k, Resistor_THT:R_Axial_DIN0204_L3.6mm_D1.6mm_P7.62mm_Horizontal, symbol Device:R
- C10, C11, C12, C13, C14, C15, C16, C17, C18, C19, C20, C5, C6, C7, C8, C9: footprint Capacitor_THT:C_Axial_L12.0mm_D6.5mm_P15.00mm_Horizontal -> Capacitor_THT:C_Disc_D10.5mm_W5.0mm_P10.00mm
- H1, H2, H3, H4: footprint MountingHole:MountingHole_3.2mm_M3 -> MountingHole:MountingHole_3.2mm_M3_DIN965_Pad
- U8: footprint Connector_PinHeader_1.00mm:PinHeader_1x16_P1.00mm_Horizontal -> Connector_PinHeader_2.54mm:PinHeader_1x16_P2.54mm_Horizontal
Connections:
- net 5V: now also C7.2, X1.4, R4.2, R5.2; no longer C7.1, X1.1
- net GND: now also C7.1, X1.1; no longer C7.2, X1.4
- net IRQ: now also R4.1, R5.1
Other:
- moved on the sheet: C7, X1

Commit message: fix Footprint for caps
were 10mm pitch, now they're 5mm pitch.

Signed-off-by: Lucy Mielke <user@domain.tld>
Parts:
- C10, C11, C12, C13, C14, C15, C16, C17, C18, C19, C20, C5, C6, C7, C8, C9: footprint Capacitor_THT:C_Disc_D10.5mm_W5.0mm_P10.00mm -> Capacitor_THT:C_Disc_D4.3mm_W1.9mm_P5.00mm
Changed lines of the file:
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@@
 			)
 		)
-		(property "Footprint" "Capacitor_THT:C_Disc_D10.5mm_W5.0mm_P10.00mm"
+		(property "Footprint" "Capacitor_THT:C_Disc_D4.3mm_W1.9mm_P5.00mm"
 			(at 33.3248 22.86 0)
 			(hide yes)
@@
 			)
 		)
-		(property "Footprint" "Capacitor_THT:C_Disc_D10.5mm_W5.0mm_P10.00mm"
+		(property "Footprint" "Capacitor_THT:C_Disc_D4.3mm_W1.9mm_P5.00mm"
 			(at 99.3648 21.59 0)
 			(hide yes)
@@
 			)
 		)
-		(property "Footprint" "Capacitor_THT:C_Disc_D10.5mm_W5.0mm_P10.00mm"
+		(property "Footprint" "Capacitor_THT:C_Disc_D4.3mm_W1.9mm_P5.00mm"
 			(at 43.18 106.9848 0)
 			(hide yes)
@@
 			)
 		)
-		(property "Footprint" "Capacitor_THT:C_Disc_D10.5mm_W5.0mm_P10.00mm"
+		(property "Footprint" "Capacitor_THT:C_Disc_D4.3mm_W1.9mm_P5.00mm"
 			(at 127 32.0548 0)
 			(hide yes)
@@
 			)
 		)
-		(property "Footprint" "Capacitor_THT:C_Disc_D10.5mm_W5.0mm_P10.00mm"
+		(property "Footprint" "Capacitor_THT:C_Disc_D4.3mm_W1.9mm_P5.00mm"
 			(at 172.72 73.9648 0)
 			(hide yes)
@@
 			)
 		)
-		(property "Footprint" "Capacitor_THT:C_Disc_D10.5mm_W5.0mm_P10.00mm"
+		(property "Footprint" "Capacitor_THT:C_Disc_D4.3mm_W1.9mm_P5.00mm"
 			(at 246.0752 127 0)
 			(hide yes)
@@
 			)
 		)
-		(property "Footprint" "Capacitor_THT:C_Disc_D10.5mm_W5.0mm_P10.00mm"
+		(property "Footprint" "Capacitor_THT:C_Disc_D4.3mm_W1.9mm_P5.00mm"
 			(at 191.4652 111.76 0)
 			(hide yes)
@@
 			)
 		)
-		(property "Footprint" "Capacitor_THT:C_Disc_D10.5mm_W5.0mm_P10.00mm"
+		(property "Footprint" "Capacitor_THT:C_Disc_D4.3mm_W1.9mm_P5.00mm"
 			(at 85.09 108.2548 0)
 			(hide yes)
@@
 			)
 		)
-		(property "Footprint" "Capacitor_THT:C_Disc_D10.5mm_W5.0mm_P10.00mm"
+		(property "Footprint" "Capacitor_THT:C_Disc_D4.3mm_W1.9mm_P5.00mm"
 			(at 243.5352 138.43 0)
 			(hide yes)
@@
 			)
 		)
-		(property "Footprint" "Capacitor_THT:C_Disc_D10.5mm_W5.0mm_P10.00mm"
+		(property "Footprint" "Capacitor_THT:C_Disc_D4.3mm_W1.9mm_P5.00mm"
 			(at 245.4148 29.21 0)
 			(hide yes)
@@
 			)
 		)
-		(property "Footprint" "Capacitor_THT:C_Disc_D10.5mm_W5.0mm_P10.00mm"
+		(property "Footprint" "Capacitor_THT:C_Disc_D4.3mm_W1.9mm_P5.00mm"
 			(at 38.4048 48.26 0)
 			(hide yes)
@@
 			)
 		)
-		(property "Footprint" "Capacitor_THT:C_Disc_D10.5mm_W5.0mm_P10.00mm"
+		(property "Footprint" "Capacitor_THT:C_Disc_D4.3mm_W1.9mm_P5.00mm"
 			(at 224.79 89.2048 0)
 			(hide yes)
@@
 			)
 		)
-		(property "Footprint" "Capacitor_THT:C_Disc_D10.5mm_W5.0mm_P10.00mm"
+		(property "Footprint" "Capacitor_THT:C_Disc_D4.3mm_W1.9mm_P5.00mm"
 			(at 212.3948 17.78 0)
 			(hide yes)
@@
 			)
 		)
-		(property "Footprint" "Capacitor_THT:C_Disc_D10.5mm_W5.0mm_P10.00mm"
+		(property "Footprint" "Capacitor_THT:C_Disc_D4.3mm_W1.9mm_P5.00mm"
 			(at 239.7252 111.76 0)
 			(hide yes)
@@
 			)
 		)
-		(property "Footprint" "Capacitor_THT:C_Disc_D10.5mm_W5.0mm_P10.00mm"
+		(property "Footprint" "Capacitor_THT:C_Disc_D4.3mm_W1.9mm_P5.00mm"
 			(at 137.4648 111.76 0)
 			(hide yes)
@@
 			)
 		)
-		(property "Footprint" "Capacitor_THT:C_Disc_D10.5mm_W5.0mm_P10.00mm"
+		(property "Footprint" "Capacitor_THT:C_Disc_D4.3mm_W1.9mm_P5.00mm"
 			(at 129.54 104.4448 0)
 			(hide yes)
